File: pcb/esp32-modbus/esp32-modbus.kicad_pcb (KiCad board)
At the start: 2 copper layers, 64.4 x 48 mm, 25 parts, among them J1 Conn_01x01_Male, J2 Conn_01x05_Male, J3 Conn_01x01_Male, J4 Conn_01x01_Male, J5 Conn_01x01_Male, Q1 2N3055, Q2 2N3055, U1 ESP32-WROOM-32U

Commit message: pcb prototype
Parts:
- removed REF**: SolderWire-0.75sqmm_1x01_D1.25mm_OD3.5mm, Connector_Wire:SolderWire-0.75sqmm_1x01_D1.25mm_OD3.5mm
- added D4: LED, LED_SMD:LED_1206_3216Metric_ReverseMount_Hole1.8x2.4mm, B.Cu at (171.5, 71.1)
- added J10: Conn_01x01_Male, custom:TestPoint_Pad_4.0x4.0mm, F.Cu at (144.9, 136.0)
- added J11: Conn_01x01_Male, Connector_PinHeader_1.00mm:PinHeader_1x01_P1.00mm_Vertical, F.Cu at (173.3, 65.4)
- added J12: Conn_01x01_Male, custom:TestPoint_Pad_4.0x4.0mm, F.Cu at (145.0, 129.6)
- added J13: Conn_01x01_Male, custom:TestPoint_Pad_4.0x4.0mm, F.Cu at (148.8, 129.7)
- added J14: Conn_01x01_Male, Connector_PinHeader_1.00mm:PinHeader_1x01_P1.00mm_Vertical, F.Cu at (169.3, 65.4)
- added J15: Conn_01x01_Male, Connector_PinHeader_1.00mm:PinHeader_1x01_P1.00mm_Horizontal, F.Cu at (173.3, 85.1)
- added J16: Conn_01x01_Male, Connector_PinHeader_1.00mm:PinHeader_1x01_P1.00mm_Vertical, F.Cu at (165.3, 65.4)
- added J17: Conn_01x01_Male, Connector_PinHeader_1.00mm:PinHeader_1x01_P1.00mm_Horizontal, F.Cu at (167.3, 85.1)
- added J18: Conn_01x01_Male, Connector_PinHeader_1.00mm:PinHeader_1x01_P1.00mm_Vertical, F.Cu at (171.3, 65.4)
- added J19: Conn_01x01_Male, Connector_PinHeader_1.00mm:PinHeader_1x01_P1.00mm_Horizontal, F.Cu at (171.3, 85.1)
- added J20: Conn_01x01_Male, Connector_PinHeader_1.00mm:PinHeader_1x01_P1.00mm_Vertical, F.Cu at (167.3, 65.4)
- added J21: Conn_01x01_Male, Connector_PinHeader_1.00mm:PinHeader_1x01_P1.00mm_Horizontal, F.Cu at (169.3, 85.1)
- added J22: Conn_01x01_Male, custom:TestPoint_Pad_4.0x4.0mm, F.Cu at (194.8, 129.6)
- added J23: Conn_01x01_Male, custom:TestPoint_Pad_4.0x4.0mm, F.Cu at (192.2, 129.7)
- added J24: Conn_01x01_Male, custom:TestPoint_Pad_4.0x4.0mm, F.Cu at (189.7, 129.7)
- added J25: Conn_01x01_Male, custom:TestPoint_Pad_4.0x4.0mm, F.Cu at (187.2, 129.7)
- added J26: Conn_01x01_Male, custom:TestPoint_Pad_4.0x4.0mm, F.Cu at (184.7, 129.7)
- added J27_VCC1: Conn_01x01_Male, custom:TestPoint_Pad_4.0x4.0mm, F.Cu at (184.7, 135.8)
- added J28_RO1: Conn_01x01_Male, custom:TestPoint_Pad_4.0x4.0mm, F.Cu at (194.7, 135.9)
- added J29_DI1: Conn_01x01_Male, custom:TestPoint_Pad_4.0x4.0mm, F.Cu at (192.2, 135.8)
- added J30_RE/DE1: Conn_01x01_Male, custom:TestPoint_Pad_4.0x4.0mm, F.Cu at (189.7, 135.8)
- added J31_GND1: Conn_01x01_Male, custom:TestPoint_Pad_4.0x4.0mm, F.Cu at (187.2, 135.8)
- added J6: Screw_Terminal_01x02, Connector:JWT_A3963_1x02_P3.96mm_Vertical, F.Cu at (134.8, 138.3)
- added J8: Conn_01x01_Male, Connector_PinHeader_1.00mm:PinHeader_1x01_P1.00mm_Horizontal, F.Cu at (165.3, 85.1)
- added J9: Conn_01x01_Male, custom:TestPoint_Pad_4.0x4.0mm, F.Cu at (148.8, 136.0)
- added JP3: SolderJumper_2_Open, Jumper:SolderJumper-2_P1.3mm_Open_Pad1.0x1.5mm, F.Cu at (187.9, 100.3)
- added R2.5k4: R, Resistor_SMD:R_0805_2012Metric_Pad1.20x1.40mm_HandSolder, F.Cu at (169.4, 88.2)
- D1, D2, D3: moved to B.Cu
- J1, J3, J4, J5: footprint Connector_Pin:Pin_D1.0mm_L10.0mm -> Connector_PinHeader_1.00mm:PinHeader_1x01_P1.00mm_Vertical
- moved Q2 170.7 mm to (187.5, 88.3), turned to 180 degrees
- moved JP2 167.7 mm to (200.2, 127.3), turned to -90 degrees
- moved J1 160.3 mm to (194.2, 89.8), turned to -90 degrees
- moved C3 159.4 mm to (172.1, 97.2), turned to 180 degrees
- moved C1 156.2 mm to (178.5, 115.1), turned to 90 degrees
- moved J5 154.2 mm to (191.7, 96.2)
- moved C4 153.2 mm to (172.1, 102.5), turned to 180 degrees
- moved R10k2 147.6 mm to (191.9, 88.6), turned to -90 degrees
- moved D3 137.3 mm to (167.8, 71.1), turned to 90 degrees
- moved JP1 136.5 mm to (191.8, 100.3)
- moved Q1 135.8 mm to (187.5, 92.7), turned to 180 degrees
- moved R10k1 133.4 mm to (183.8, 100.4)
- moved C2 130.6 mm to (180.8, 115.1), turned to 90 degrees
- moved J4 129.4 mm to (194.1, 96.2)
- moved D1 113.4 mm to (164.2, 71.1), turned to 90 degrees
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Connections:
- D1 pad 2: /GPIO2 -> Net-(D1-Pad2)
- D2 pad 1: Net-(D2-Pad1) -> Net-(D1-Pad1)
- D2 pad 2: /TX -> Net-(D2-Pad2)
- D3 pad 1: Net-(D3-Pad1) -> Net-(D1-Pad1)
- D3 pad 2: /RX -> Net-(D3-Pad2)
- J2 pad 1: GND -> Net-(J2-Pad1)
- J2 pad 2: /GPIO2 -> Net-(J2-Pad2)
- J2 pad 3: /TX -> Net-(J2-Pad3)
- J2 pad 4: /RX -> Net-(J2-Pad4)
- J2 pad 5: +3.3V -> Net-(J2-Pad5)
- PS1 pad 1: unconnected-(PS1-Pad1) -> Net-(J12-Pad1)
- PS1 pad 2: unconnected-(PS1-Pad2) -> Net-(J13-Pad1)
- R10k1 pad 2: /EN -> Net-(JP3-Pad1)
- R2.5k1 pad 1: Net-(D1-Pad1) -> +3.3V
- R2.5k1 pad 2: GND -> Net-(J15-Pad1)
- R2.5k2 pad 1: Net-(D2-Pad1) -> /GPIO2
- R2.5k2 pad 2: GND -> Net-(J17-Pad1)
- R2.5k3 pad 1: Net-(D3-Pad1) -> /TX
- R2.5k3 pad 2: GND -> Net-(J19-Pad1)
Routing:
- net GND: track 0.00 -> 81.8 mm, vias 0 -> 4
- net /TX: track 0.00 -> 61.4 mm, vias 0 -> 2
- net /GPIO0: track 0.00 -> 60.6 mm, vias 0 -> 2
- net /GPIO2: track 0.00 -> 59.2 mm, vias 0 -> 2
- net +3.3V: track 0.00 -> 58.1 mm
- net /RX: track 0.00 -> 58.1 mm, vias 0 -> 2
- net Net-(D1-Pad1): track 0.00 -> 23.6 mm
- net /RXP: track 0.00 -> 22.7 mm
- net /TXD: track 0.00 -> 21.8 mm
- net /EN: track 0.00 -> 19.8 mm
- net Net-(J2-Pad5): track 0.00 -> 19.7 mm, vias 0 -> 1
- net Net-(J6-Pad2): track 0.00 -> 19.4 mm
- net Net-(J12-Pad1): track 0.00 -> 18.9 mm
- net Net-(J2-Pad1): track 0.00 -> 14.8 mm
- net Net-(J13-Pad1): track 0.00 -> 12.9 mm
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Other:
- board size 64.4 x 48 mm -> 85.8 x 83.4 mm
